File: KiCad/Sheet_a.kicad_sch (KiCad schematic)
At the start: 0 parts

Commit message: Alimentcaio
Parts:
- added C? (x2): 10 uF, symbol Device:C_US
- added D?: 1N4007, Diode_THT:D_DO-41_SOD81_P10.16mm_Horizontal, symbol Diode:1N4007
- added J?: Conn_01x01_Pin, symbol Connector:Conn_01x01_Pin
- added U?: LM2596S-5, Package_TO_SOT_SMD:TO-263-5_TabPin3, symbol Regulator_Switching:LM2596S-5
- added U?: LM1117DT-3.3, Package_TO_SOT_SMD:TO-252-3_TabPin2, symbol Regulator_Linear:LM1117DT-3.3
Connections:
- new net: C?.1, D?.1 (K), U?.2 (OUT), U?.3 (VI), U?.4 (FB)
- new net GND: C?.2, C?.2, D?.2 (A), U?.1 (GND), U?.3 (GND), U?.5 (~{ON}/OFF)
- new net VBAT: J?.1 (Pin_1), U?.1 (VIN)
- new net VCC: C?.1, U?.2 (VO)
Other:
- note added: "Alimentació"
