File: KiCad/Sheet_f.kicad_sch (KiCad schematic)
At the start: 0 parts

Commit message: Microchip afegit
Parts:
- added C5, C6: 33pF, Capacitor_SMD:C_0805_2012Metric, symbol Device:C
- added U4: Pic24hj128gp502, Package_SO:SOIC-28W_7.5x17.9mm_P1.27mm, symbol simbolo:Pic24hj128gp502
- added Y?: Crystal, Crystal:Crystal_HC49-U_Vertical, symbol Device:Crystal
Connections:
- new net GND: C5.2, C6.2, U4.16 (VSS), U4.5 (Vss)
- new net OSC1: C5.1, U4.6 (RA2/OSC1), Y?.1
- new net OSC2: C6.1, U4.7 (RA3/OSC2), Y?.2
- new net VCC: U4.10 (VDD)
Other:
- note added: "OSCILATOR"
