File: KiCad/POTENCIA.kicad_sch (KiCad schematic)
At the start: 15 parts, among them J3 Conn_01x02_Pin, J7 Conn_01x02_Pin, J8 Conn_01x02_Pin, SW7 SW_SPST, U2 LM2596S-5, U3 L298N, U7 LM1117DT-3.3

Commit message: Pequeño error
Other:
- note added: "Motor1+"
- note added: "Motor1-"
- note added: "Motor2+"
- note added: "Motor2-"
- note removed: "Motor+"
- note removed: "Motor-"
Changed lines of the file:
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@@
 		)
 	)
-	(text "Motor-"
+	(text "Motor2-"
 		(exclude_from_sim no)
 		(at 78.232 150.368 0)
@@
 		)
 	)
-	(text "Motor+"
+	(text "Motor1+"
 		(exclude_from_sim no)
 		(at 77.978 139.954 0)
@@
 		)
 	)
-	(text "Motor+"
+	(text "Motor2+"
 		(exclude_from_sim no)
 		(at 78.232 147.574 0)
@@
 		)
 	)
-	(text "Motor-"
+	(text "Motor1-"
 		(exclude_from_sim no)
 		(at 77.978 142.748 0)
