File: KiCad/Grup_D_Llums.kicad_pcb (KiCad board)
At the start: 2 copper layers, 89 parts, among them J1 DE9_Pins, J2 Screw_Terminal_01x02, J3 Screw_Terminal_01x02, J4 Conn_PIC_ICSP_ICD, J5 DE9_Pins, J6 Screw_Terminal_01x02, J7 Conn_01x10_Pin, Q1 AO3400A, Q2 AO3400A, Q3 AO3400A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

Commit message: Placa
Parts:
- added REF**: MountingHole_2.2mm_M2, MountingHole:MountingHole_2.2mm_M2, F.Cu at (88.0, 46.1)
- added REF**: MountingHole_2.2mm_M2, MountingHole:MountingHole_2.2mm_M2, F.Cu at (187.4, 46.0)
- added REF**: MountingHole_2.2mm_M2, MountingHole:MountingHole_2.2mm_M2, F.Cu at (187.1, 146.6)
- added REF**: MountingHole_2.2mm_M2, MountingHole:MountingHole_2.2mm_M2, F.Cu at (88.5, 146.6)
- moved J1 161.4 mm to (178.5, 125.0), turned to 90 degrees
- moved SW4 157.7 mm to (162.5, 126.9)
- moved SW2 157.6 mm to (143.9, 129.6), turned to 90 degrees
- moved SW3 154.9 mm to (149.3, 129.6), turned to 90 degrees
- moved SW5 148.4 mm to (163.4, 117.2), turned to 90 degrees
- moved J7 138.3 mm to (159.8, 54.4)
- moved C7 137.4 mm to (155.5, 145.2)
- moved C3 136.7 mm to (163.1, 134.9)
- moved C6 136.1 mm to (148.7, 145.1), turned to 180 degrees
- moved R12 129.2 mm to (166.1, 137.2), turned to 90 degrees
- moved J5 128.0 mm to (178.7, 85.3), turned to 90 degrees
- moved R13 126.3 mm to (164.1, 138.1), turned to -90 degrees
- moved SW6 125.1 mm to (134.4, 129.8)
- moved Q4 124.5 mm to (145.9, 44.8), turned to 90 degrees
- moved SW1 122.0 mm to (145.7, 122.8), turned to 180 degrees
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Connections:
- J5 pad 2: Net-(U1-RA9) -> Usart1
- J7 pad 2: LOW_L -> HI_L
- J7 pad 3: LOW_R -> HI_R
- J7 pad 4: HI_L -> LOW_L
- J7 pad 5: HI_R -> LOW_R
- U1 pad 1: SDA -> DRL_CTRL
- U1 pad 11: LF_REV -> unconnected-(U1-RB13-Pad11)
- U1 pad 13: LIGHT_INT -> unconnected-(U1-RA7-Pad13)
- U1 pad 15: unconnected-(U1-RB15-Pad15) -> IN_LF
- U1 pad 2: DRL_CTRL -> TURN_LEFT_CTRL
- U1 pad 3: TURN_LEFT_CTRL -> TURN_RIGHT_CTRL
- U1 pad 33: unconnected-(U1-RB4-Pad33) -> Usart1
- U1 pad 34: unconnected-(U1-RA4-Pad34) -> LF_LIMIT
- U1 pad 35: Net-(U1-RA9) -> unconnected-(U1-RA9-Pad35)
- U1 pad 36: IN_LF -> unconnected-(U1-RC3-Pad36)
- U1 pad 37: LF_LIMIT -> unconnected-(U1-RC4-Pad37)
- U1 pad 38: unconnected-(U1-RC5-Pad38) -> SCL
- U1 pad 4: TURN_RIGHT_CTRL -> LOW_BEAM_CTRL
- U1 pad 43: unconnected-(U1-RB7-Pad43) -> SDA
- U1 pad 44: SCL -> LIGHT_INT
- U1 pad 5: LOW_BEAM_CTRL -> HI_BEAM_CTRL
- U1 pad 8: HI_BEAM_CTRL -> LF_FWD
- U1 pad 9: LF_FWD -> LF_REV
Routing:
- net VCC: track 16.9 -> 143.0 mm
- net HI_BEAM_CTRL: track 0.00 -> 76.0 mm
- net LOW_BEAM_CTRL: track 0.00 -> 60.9 mm
- net TURN_RIGHT_CTRL: track 0.00 -> 43.1 mm
- net 5VOLTS: track 0.00 -> 36.1 mm
- net TURN_LEFT_CTRL: track 0.00 -> 35.8 mm
- net Usart1: track 0.00 -> 35.2 mm
- net Net-(U1-RA8): track 0.00 -> 34.2 mm
- net DRL_CTRL: track 0.00 -> 31.8 mm
- net RXD: track 0.00 -> 27.9 mm
- net Net-(U6-CANH): track 0.00 -> 26.4 mm
- net HI_L: track 0.00 -> 24.5 mm
- net DRL_O: track 0.00 -> 22.7 mm
- net Net-(U6-CANL): track 0.00 -> 21.6 mm
- net Net-(D3-K): track 0.00 -> 21.1 mm
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- added copper zone on B.Cu, net GND
- added copper zone on F.Cu, net GND
- added copper zone on F.Cu, net VCC

Commit message: Hello
Parts:
- moved J3 30.1 mm to (90.4, 97.9), turned to 90 degrees
Routing:
- net Net-(D5-A): track 22.7 -> 40.7 mm
- net Net-(D11-A): track 30.4 -> 47.9 mm
Other:
- board text removed: "ALIMENTACIO"
- board text removed: "DRIVER MOTOR"
Changed lines of the file:
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@@
 	(footprint "TerminalBlock_Phoenix:TerminalBlock_Phoenix_MKDS-1,5-2-5.08_1x02_P5.08mm_Horizontal"
 		(layer "F.Cu")
-		(at 120.507831 98.6075)
+		(at 90.3725 97.895 90)
 		(descr "Terminal Block Phoenix MKDS-1,5-2-5.08, 2 pins, pitch 5.08mm, size 10.2x9.8mm, drill diameter 1.3mm, pad diameter 2.6mm, http://www.farnell.com/datasheets/100425.pdf, script-generated using https://gitlab.com/kicad/libraries/kicad-footprint-generator/-/tree/master/scripts/TerminalBlock_Phoenix")
 		(tags "THT Terminal Block Phoenix MKDS-1,5-2-5.08 pitch 5.08mm size 10.2x9.8mm drill 1.3mm pad 2.6mm")
 		(property "Reference" "J3"
-			(at 2.54 -6.32 0)
+			(at 2.54 -6.32 90)
 			(layer "F.SilkS")
 			(effects
@@
 		)
 		(property "Value" "Screw_Terminal_01x02"
-			(at 2.54 5.72 0)
+			(at 2.54 5.72 90)
 			(layer "F.Fab")
 			(effects
@@
 		)
 		(property "Datasheet" "~"
-			(at 0 0 0)
+			(at 0 0 90)
 			(layer "F.Fab")
 			(hide yes)
@@
 		)
 		(property "Description" "Generic screw terminal, single row, 01x02, script generated (kicad-library-utils/schlib/autogen/connector/)"
-			(at 0 0 0)
+			(at 0 0 90)
 			(layer "F.Fab")
 			(hide yes)
@@
 		(attr through_hole)
 		(fp_line
+			(start 7.74 -5.32)
+			(end 7.74 4.72)
+			(stroke
+				(width 0.12)
+				(type solid)
+			)
+			(layer "F.SilkS")
+		)
+		(fp_line
 			(start -2.66 -5.32)
 			(end 7.74 -5.32)
@@
 		)
 		(fp_line
-			(start -2.66 4.72)
-			(end -2.66 -5.32)
+			(start 7.74 4.72)
+			(end 0.3 4.72)
 			(stroke
 				(width 0.12)
@@
 		)
 		(fp_line
-			(start 7.74 -5.32)
-			(end 7.74 4.72)
-			(stroke
-				(width 0.12)
-				(type solid)
-			)
-			(layer "F.SilkS")
-		)
-		(fp_line
-			(start 7.74 4.72)
-			(end 0.3 4.72)
+			(start -2.66 4.72)
+			(end -2.66 -5.32)
 			(stroke
 				(width 0.12)
@@
 		)
 		(fp_line
-			(start -2.54 -5.2)
-			(end 7.62 -5.2)
+			(start 7.62 -5.2)
+			(end 7.62 4.6)
 			(stroke
 				(width 0.1)
@@
 		)
 		(fp_line
-			(start -2.54 -2.3)
-			(end 7.62 -2.3)
+			(start -2.54 -5.2)
+			(end 7.62 -5.2)
 			(stroke
 				(width 0.1)
@@
 		)
 		(fp_line
-			(start -2.54 2.6)
-			(end 7.62 2.6)
+			(start -2.54 -2.3)
+			(end 7.62 -2.3)
 			(stroke
 				(width 0.1)
@@
 		)
 		(fp_line
-			(start -2.54 4.1)
-			(end -2.54 -5.2)
+			(start 6.035 -1.138)
+			(end 3.942 0.955)
 			(stroke
 				(width 0.1)
@@
 		)
 		(fp_line
-			(start -2.54 4.1)
-			(end 7.62 4.1)
+			(start 0.955 -1.138)
+			(end -1.138 0.955)
 			(stroke
 				(width 0.1)
@@
 		)
 		(fp_line
-			(start -2.04 4.6)
-			(end -2.54 4.1)
+			(start 6.218 -0.955)
+			(end 4.125 1.138)
 			(stroke
 				(width 0.1)
@@
 		)
 		(fp_line
-			(start 0.955 -1.138)
-			(end -1.138 0.955)
+			(start 1.138 -0.955)
+			(end -0.955 1.138)
 			(stroke
 				(width 0.1)
@@
 		)
 		(fp_line
-			(start 1.138 -0.955)
-			(end -0.955 1.138)
+			(start -2.54 2.6)
+			(end 7.62 2.6)
 			(stroke
 				(width 0.1)
@@
 		)
 		(fp_line
-			(start 6.035 -1.138)
-			(end 3.942 0.955)
+			(start -2.54 4.1)
+			(end -2.54 -5.2)
 			(stroke
 				(width 0.1)
@@
 		)
 		(fp_line
-			(start 6.218 -0.955)
-			(end 4.125 1.138)
+			(start -2.54 4.1)
+			(end 7.62 4.1)
 			(stroke
 				(width 0.1)
@@
 		)
 		(fp_line
-			(start 7.62 -5.2)
-			(end 7.62 4.6)
+			(start 7.62 4.6)
+			(end -2.04 4.6)
 			(stroke
 				(width 0.1)
@@
 		)
 		(fp_line
-			(start 7.62 4.6)
-			(end -2.04 4.6)
+			(start -2.04 4.6)
+			(end -2.54 4.1)
 			(stroke
 				(width 0.1)
@@
 		)
 		(fp_circle
-			(center 0 0)
-			(end 1.5 0)
+			(center 5.08 0)
+			(end 6.58 0)
 			(stroke
 				(width 0.1)
@@
 		)
 		(fp_circle
-			(center 5.08 0)
-			(end 6.58 0)
+			(center 0 0)
+			(end 1.5 0)
 			(stroke
 				(width 0.1)
@@
 		)
 		(fp_text user "${REFERENCE}"
-			(at 2.54 3.2 0)
+			(at 2.54 3.2 90)
 			(layer "F.Fab")
 			(effects
@@
 		)
 		(pad "1" thru_hole roundrect
-			(at 0 0)
+			(at 0 0 90)
 			(size 2.6 2.6)
 			(drill 1.3)
@@
 		)
 		(pad "2" thru_hole circle
-			(at 5.08 0)
+			(at 5.08 0 90)
 			(size 2.6 2.6)
 			(drill 1.3)
@@
 		)
 	)
-	(gr_text "DRIVER MOTOR"
-		(at 99.882831 104.285 0)
-		(layer "F.Cu")
-		(effects
-			(font
-				(size 1.5 1.5)
-				(thickness 0.3)
-				(bold yes)
-			)
-			(justify left bottom)
-		)
-	)
-	(gr_text "ALIMENTACIO"
-		(at 89.325331 56.885 0)
-		(layer "F.Cu")
-		(effects
-			(font
-				(size 1.5 1.5)
-				(thickness 0.3)
-				(bold yes)
-			)
-			(justify left bottom)
-		)
-	)
 	(via
 		(at 174.625331 106.585)
@@
 	)
 	(segment
+		(start 90.3725 97.895)
+		(end 94.5775 102.1)
+		(width 0.2)
+		(layer "F.Cu")
+		(net 13)
+	)
+	(segment
 		(start 113.652831 114.285)
 		(end 113.652831 108.115)
@@
 	)
 	(segment
-		(start 120.442831 107.985)
-		(end 120.502831 107.925)
+		(start 107.637831 102.1)
+		(end 113.522831 107.985)
 		(width 0.2)
 		(layer "F.Cu")
@@
 	)
 	(segment
-		(start 113.652831 108.115)
-		(end 113.522831 107.985)
+		(start 120.442831 107.985)
+		(end 120.502831 107.925)
 		(width 0.2)
 		(layer "F.Cu")
@@
 	)
 	(segment
-		(start 120.507831 98.6075)
-		(end 120.507831 107.92)
+		(start 94.5775 102.1)
+		(end 107.637831 102.1)
 		(width 0.2)
 		(layer "F.Cu")
@@
 	)
 	(segment
-		(start 115.152831 98.805)
-		(end 115.122831 98.835)
+		(start 113.652831 108.115)
+		(end 113.522831 107.985)
 		(width 0.2)
 		(layer "F.Cu")
-		(net 14)
+		(net 13)
 	)
 	(segment
-		(start 125.582831 109.195)
-		(end 127.092831 107.685)
+		(start 90.3725 92.815)
+		(end 92.9375 90.25)
 		(width 0.2)
 		(layer "F.Cu")
@@
 	)
 	(segment
-		(start 123.715331 96.735)
-		(end 125.587831 98.6075)
+		(start 115.152831 98.805)
+		(end 115.122831 98.835)
 		(width 0.2)
 		(layer "F.Cu")
@@
 	)
 	(segment
-		(start 127.092831 107.685)
-		(end 127.092831 100.1125)
+		(start 115.122831 98.835)
+		(end 125.482831 109.195)
 		(width 0.2)
 		(layer "F.Cu")
@@
 	)
 	(segment
-		(start 115.152831 92.435)
-		(end 115.152831 98.805)
+		(start 125.482831 109.195)
+		(end 125.582831 109.195)
 		(width 0.2)
 		(layer "F.Cu")
@@
 	)
 	(segment
-		(start 117.222831 96.735)
-		(end 123.715331 96.735)
+		(start 112.967831 90.25)
+		(end 115.152831 92.435)
 		(width 0.2)
 		(layer "F.Cu")
@@
 	)
 	(segment
-		(start 127.092831 100.1125)
-		(end 125.587831 98.6075)
+		(start 92.9375 90.25)
+		(end 112.967831 90.25)
 		(width 0.2)
 		(layer "F.Cu")
@@
 	)
 	(segment
-		(start 115.122831 98.835)
-		(end 117.222831 96.735)
+		(start 115.152831 92.435)
+		(end 115.152831 98.805)
 		(width 0.2)
 		(layer "F.Cu")
@@
 	)
 	(zone
-		(net 0)
-		(net_name "")
-		(layer "F.Cu")
-		(hatch edge 0.5)
-		(connect_pads
-			(clearance 0)
-		)
-		(min_thickness 0.25)
-		(filled_areas_thickness no)
-		(keepout
-			(tracks not_allowed)
-			(vias not_allowed)
-			(pads not_allowed)
-			(copperpour allowed)
-			(footprints allowed)
-		)
-		(placement
-			(enabled no)
-			(sheetname "/LLUMS/")
-		)
-		(fill
-			(thermal_gap 0.5)
-			(thermal_bridge_width 0.5)
-		)
-		(polygon
-			(pts
-				(xy 83.844143 42.502975) (xy 192.344143 42.202975) (xy 192.044143 150.302975) (xy 83.544143 150.602975)
-			)
-		)
-	)
-	(zone

Commit message: PCB Hotfixes
Parts:
- moved R8 1.99 mm to (144.4, 47.9), turned to 0 degrees
- moved C2 1.44 mm to (142.9, 105.2), turned to 180 degrees
Routing:
- net GND: track 0.00 -> 160.4 mm, vias 204 -> 297
- net MCLR: track 8.20 -> 12.9 mm
- net Net-(U1-VBUS): track 0.00 -> 3.37 mm
- net LIGHT_INT: track 12.0 -> 13.5 mm

Commit message: R
Parts:
- removed the REF** at (88.0, 46.1)
- removed the REF** at (187.4, 46.0)
- removed the REF** at (187.1, 146.6)
- removed the REF** at (88.5, 146.6)
- added REF**: MountingHole_2.2mm_M2, MountingHole:MountingHole_2.2mm_M2, F.Cu at (74.3, 142.0)
- added REF**: MountingHole_2.2mm_M2, MountingHole:MountingHole_2.2mm_M2, F.Cu at (196.7, 38.4)
- added REF**: MountingHole_2.2mm_M2, MountingHole:MountingHole_2.2mm_M2, F.Cu at (97.3, 38.5)
- added REF**: MountingHole_2.2mm_M2, MountingHole:MountingHole_2.2mm_M2, F.Cu at (196.4, 139.0)
- U3: moved to F.Cu
- moved J2 55.8 mm to (137.4, 43.8), turned to 180 degrees
- moved F4 51.5 mm to (171.9, 86.1), turned to 0 degrees
- moved R7 48.3 mm to (171.9, 84.1), turned to 180 degrees
- moved D7 46.5 mm to (134.4, 129.9), turned to 180 degrees
- moved Q4 46.2 mm to (168.4, 85.2), turned to -90 degrees
- moved R8 43.9 mm to (171.9, 82.1)
- moved F7 42.3 mm to (171.9, 80.1), turned to 0 degrees
- moved C1 41.2 mm to (94.4, 77.8), turned to 180 degrees
- moved R17 39.5 mm to (171.9, 78.1), turned to 180 degrees
- moved C10 39.4 mm to (93.3, 71.8), turned to 180 degrees
- moved R18 36.9 mm to (171.9, 76.1), turned to 0 degrees
- moved Q7 36.3 mm to (168.5, 79.2), turned to -90 degrees
- moved F8 33.2 mm to (171.9, 72.6), turned to 0 degrees
- moved D11 32.2 mm to (119.2, 118.2)
- moved R19 31.6 mm to (171.9, 70.6), turned to 180 degrees
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Connections:
- D6 pad 1: GND -> VCC
- D6 pad 2: Net-(D5-A) -> Net-(D11-A)
- D7 pad 2: Net-(D11-A) -> Net-(D10-A)
- D9 pad 1: VCC -> GND
- D9 pad 2: Net-(D10-A) -> Net-(D5-A)
- J7 pad 2: HI_L -> LOW_R
- J7 pad 3: HI_R -> LOW_L
- J7 pad 4: LOW_L -> HI_R
- J7 pad 5: LOW_R -> HI_L
- U1 pad 12: LF_PWM -> LF_FWD
- U1 pad 8: LF_FWD -> LF_PWM
Routing:
- net GND: track 160.4 -> 0.00 mm, vias 297 -> 204
- net VBAT: track 8.36 -> 104.8 mm
- net Net-(D11-A): track 47.9 -> 132.5 mm
- net LF_REV: track 16.6 -> 47.5 mm
- net LF_FWD: track 17.3 -> 47.5 mm
- net LF_PWM: track 17.5 -> 45.2 mm
- net HI_BEAM_CTRL: track 76.0 -> 103.5 mm
- net Net-(D10-A): track 45.2 -> 69.4 mm
- net LOW_BEAM_CTRL: track 60.9 -> 84.9 mm
- net Net-(D12-A): track 44.2 -> 64.9 mm
- net VCC: track 143.0 -> 162.7 mm
- net DRL_O: track 22.7 -> 10.1 mm
- net DRR_O: track 20.3 -> 11.1 mm
- net INT_L: track 18.9 -> 12.9 mm
- net MCLR: track 12.9 -> 8.20 mm
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- added copper zone on F.Cu, net VBAT
- removed copper zone on B.Cu, net GND
Other:
- board text added: "ALIMENTACIO"
- board text added: "DRIVER MOTOR"

Commit message: B, ground
Parts:
- added REF**: TestPoint_Bridge_Pitch2.0mm_Drill0.7mm, TestPoint:TestPoint_Bridge_Pitch2.0mm_Drill0.7mm, F.Cu at (139.4, 100.8)
- moved REF** 24.6 mm to (81.9, 57.7)
- moved REF** 18.9 mm to (196.6, 57.3)
- moved J2 16.3 mm to (140.2, 59.9)
- moved REF** 12.5 mm to (196.5, 151.5)
- moved REF** 12.1 mm to (81.4, 151.8)
- moved C10 12.0 mm to (93.4, 83.8)
- moved C11 12.0 mm to (112.1, 87.3)
- moved D4 12.0 mm to (112.5, 64.8)
- moved L1 12.0 mm to (103.2, 84.8)
- moved U2 12.0 mm to (121.2, 80.6)
- moved C9 12.0 mm to (107.3, 70.6)
- moved C1 12.0 mm to (94.5, 89.7)
- moved D1 12.0 mm to (108.1, 79.0)
- moved D3 12.0 mm to (112.6, 71.2)
- moved U7 12.0 mm to (113.4, 94.8)
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Routing:
- net GND: track 0.00 -> 139.2 mm, vias 204 -> 140
- net VBAT: track 104.8 -> 237.6 mm
- net VCC: track 162.7 -> 135.3 mm
- net LOW_BEAM_CTRL: track 84.9 -> 88.9 mm
- net HI_BEAM_CTRL: track 103.5 -> 106.9 mm
- net HI_L: track 22.7 -> 26.0 mm
- net INT_R: track 16.7 -> 19.7 mm
- net TURN_RIGHT_CTRL: track 43.3 -> 46.2 mm
- net DRL_O: track 10.1 -> 8.11 mm
- net Net-(Q7-G): track 3.60 -> 1.60 mm
- net INT_L: track 12.9 -> 14.8 mm
- net TURN_LEFT_CTRL: track 36.3 -> 38.2 mm
- net LOW_R: track 14.4 -> 13.0 mm
- net LOW_L: track 17.2 -> 16.0 mm
- net Net-(Q6-G): track 3.32 -> 4.32 mm
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- added copper zone on B.Cu, net GND

Commit message: grund c
Parts:
- moved REF** 1.20 mm to (139.3, 102.0), turned to 90 degrees
Routing:
- net GND: track 139.2 -> 142.7 mm, vias 140 -> 143
Changed lines of the file:
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@@
 	(footprint "TestPoint:TestPoint_Bridge_Pitch2.0mm_Drill0.7mm"
 		(layer "F.Cu")
-		(at 139.4 100.8)
+		(at 139.3 102 90)
 		(descr "wire loop as test point, pitch 2.0mm, hole diameter 0.7mm, wire diameter 0.5mm")
 		(tags "test point wire loop")
 		(property "Reference" "REF**"
-			(at 1.1 1.7 0)
+			(at 1.1 1.7 90)
 			(layer "F.SilkS")
 			(effects
@@
 		)
 		(property "Value" "TestPoint_Bridge_Pitch2.0mm_Drill0.7mm"
-			(at 1 -1.7 0)
+			(at 1 -1.7 90)
 			(layer "F.Fab")
 			(effects
@@
 		)
 		(property "Datasheet" ""
-			(at 0 0 0)
+			(at 0 0 90)
 			(unlocked yes)
 			(layer "F.Fab")
@@
 		)
 		(property "Description" ""
-			(at 0 0 0)
+			(at 0 0 90)
 			(unlocked yes)
 			(layer "F.Fab")
@@
 		(attr through_hole)
 		(fp_line
+			(start 2.9 -0.9)
+			(end -0.9 -0.9)
+			(stroke
+				(width 0.12)
+				(type solid)
+			)
+			(layer "F.SilkS")
+		)
+		(fp_line
 			(start -0.9 -0.9)
 			(end -0.9 0.9)
@@
 		)
 		(fp_line
+			(start 2.9 0.9)
+			(end 2.9 -0.9)
+			(stroke
+				(width 0.12)
+				(type solid)
+			)
+			(layer "F.SilkS")
+		)
+		(fp_line
 			(start -0.9 0.9)
 			(end 2.9 0.9)
@@
 		)
 		(fp_line
-			(start 2.9 -0.9)
-			(end -0.9 -0.9)
-			(stroke
-				(width 0.12)
-				(type solid)
-			)
-			(layer "F.SilkS")
-		)
-		(fp_line
-			(start 2.9 0.9)
-			(end 2.9 -0.9)
-			(stroke
-				(width 0.12)
-				(type solid)
-			)
-			(layer "F.SilkS")
+			(start 3.2 -1.2)
+			(end -1.2 -1.2)
+			(stroke
+				(width 0.05)
+				(type solid)
+			)
+			(layer "F.CrtYd")
+		)
+		(fp_line
+			(start 3.2 -1.2)
+			(end 3.2 1.2)
+			(stroke
+				(width 0.05)
+				(type solid)
+			)
+			(layer "F.CrtYd")
 		)
 		(fp_line
@@
 		)
 		(fp_line
-			(start 3.2 -1.2)
-			(end -1.2 -1.2)
-			(stroke
-				(width 0.05)
-				(type solid)
-			)
-			(layer "F.CrtYd")
-		)
-		(fp_line
-			(start 3.2 -1.2)
-			(end 3.2 1.2)
-			(stroke
-				(width 0.05)
-				(type solid)
-			)
-			(layer "F.CrtYd")
-		)
-		(fp_line
 			(start 2 0)
 			(end 0 0)
@@
 		)
 		(fp_text user "${REFERENCE}"
-			(at 1.1 1.7 0)
+			(at 1.1 1.7 90)
 			(layer "F.Fab")
 			(effects
@@
 		)
 		(pad "1" thru_hole circle
-			(at 0 0)
+			(at 0 0 90)
 			(size 1.4 1.4)
 			(drill 0.7)
@@
 		)
 		(pad "1" thru_hole circle
-			(at 2 0)
+			(at 2 0 90)
 			(size 1.4 1.4)
 			(drill 0.7)
@@
 	)
 	(segment
+		(start 114.85 120.95)
+		(end 113.75 120.95)
+		(width 0.2)
+		(layer "F.Cu")
+		(net 1)
+	)
+	(segment
 		(start 158.075331 93.385)
 		(end 158.075331 94.775331)
@@
 	)
 	(segment
+		(start 115.95 120.95)
+		(end 116 120.9)
+		(width 0.2)
+		(layer "F.Cu")
+		(net 1)
+	)
+	(segment
 		(start 167.5 81)
 		(end 167.5 82.3105)
@@
 	)
 	(segment
+		(start 114.85 120.95)
+		(end 115.95 120.95)
+		(width 0.2)
+		(layer "F.Cu")
+		(net 1)
+	)
+	(segment
 		(start 153.025 60.075)
 		(end 153 60.1)
@@
 	)
 	(segment
+		(start 113.75 120.95)
+		(end 113.7 120.9)
+		(width 0.2)
+		(layer "F.Cu")
+		(net 1)
+	)
+	(segment
 		(start 167.4375 61.4)
 		(end 167.4625 61.425)
@@
 	)
 	(segment
+		(start 114.85 119.85)
+		(end 114.8 119.8)
+		(width 0.2)
+		(layer "F.Cu")
+		(net 1)
+	)
+	(segment
 		(start 116.375 83.975)
 		(end 116.4 84)
@@
 	)
 	(segment
+		(start 114.85 120.95)
+		(end 114.85 119.85)
+		(width 0.2)
+		(layer "F.Cu")
+		(net 1)
+	)
+	(segment
 		(start 165.790331 137.6)
 		(end 165.775331 137.585)
@@
 	)
 	(via
+		(at 116 120.9)
+		(size 0.6)
+		(drill 0.3)
+		(layers "F.Cu" "B.Cu")
+		(free yes)
+		(net 1)
+	)
+	(via
 		(at 190 108.9)
 		(size 0.6)
@@
 		(size 0.6)
 		(drill 0.3)
+		(layers "F.Cu" "B.Cu")
+		(free yes)
+		(net 1)
+	)
+	(via
+		(at 113.7 120.9)
+		(size 0.6)
+		(drill 0.3)
+		(layers "F.Cu" "B.Cu")
+		(free yes)
+		(net 1)
+	)
+	(via
+		(at 114.8 119.8)
+		(size 0.6)
+		(drill 0.3)

Commit message: Hotfixes
Parts:
- removed the REF** at (139.3, 102.0)
Other:
- board text removed: "ALIMENTACIO"
- board text removed: "DRIVER MOTOR"
Changed lines of the file:
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@@
-		)
-	)
-	(footprint "TestPoint:TestPoint_Bridge_Pitch2.0mm_Drill0.7mm"
-		(layer "F.Cu")
-		(at 139.3 102 90)
-		(descr "wire loop as test point, pitch 2.0mm, hole diameter 0.7mm, wire diameter 0.5mm")
-		(tags "test point wire loop")
-		(property "Reference" "REF**"
-			(at 1.1 1.7 90)
-			(layer "F.SilkS")
-			(effects
-				(font
-					(size 1 1)
-					(thickness 0.15)
-				)
-			)
-		)
-		(property "Value" "TestPoint_Bridge_Pitch2.0mm_Drill0.7mm"
-			(at 1 -1.7 90)
-			(layer "F.Fab")
-			(effects
-				(font
-					(size 1 1)
-					(thickness 0.15)
-				)
-			)
-		)
-		(property "Datasheet" ""
-			(at 0 0 90)
-			(unlocked yes)
-			(layer "F.Fab")
-			(hide yes)
-			(effects
-				(font
-					(size 1.27 1.27)
-					(thickness 0.15)
-				)
-			)
-		)
-		(property "Description" ""
-			(at 0 0 90)
-			(unlocked yes)
-			(layer "F.Fab")
-			(hide yes)
-			(effects
-				(font
-					(size 1.27 1.27)
-					(thickness 0.15)
-				)
-			)
-		)
-		(attr through_hole)
-		(fp_line
-			(start 2.9 -0.9)
-			(end -0.9 -0.9)
-			(stroke
-				(width 0.12)
-				(type solid)
-			)
-			(layer "F.SilkS")
-		)
-		(fp_line
-			(start -0.9 -0.9)
-			(end -0.9 0.9)
-			(stroke
-				(width 0.12)
-				(type solid)
-			)
-			(layer "F.SilkS")
-		)
-		(fp_line
-			(start 2.9 0.9)
-			(end 2.9 -0.9)
-			(stroke
-				(width 0.12)
-				(type solid)
-			)
-			(layer "F.SilkS")
-		)
-		(fp_line
-			(start -0.9 0.9)
-			(end 2.9 0.9)
-			(stroke
-				(width 0.12)
-				(type solid)
-			)
-			(layer "F.SilkS")
-		)
-		(fp_line
-			(start 3.2 -1.2)
-			(end -1.2 -1.2)
-			(stroke
-				(width 0.05)
-				(type solid)
-			)
-			(layer "F.CrtYd")
-		)
-		(fp_line
-			(start 3.2 -1.2)
-			(end 3.2 1.2)
-			(stroke
-				(width 0.05)
-				(type solid)
-			)
-			(layer "F.CrtYd")
-		)
-		(fp_line
-			(start -1.2 1.2)
-			(end -1.2 -1.2)
-			(stroke
-				(width 0.05)
-				(type solid)
-			)
-			(layer "F.CrtYd")
-		)
-		(fp_line
-			(start -1.2 1.2)
-			(end 3.2 1.2)
-			(stroke
-				(width 0.05)
-				(type solid)
-			)
-			(layer "F.CrtYd")
-		)
-		(fp_line
-			(start 2 0)
-			(end 0 0)
-			(stroke
-				(width 0.12)
-				(type solid)
-			)
-			(layer "F.Fab")
-		)
-		(fp_text user "${REFERENCE}"
-			(at 1.1 1.7 90)
-			(layer "F.Fab")
-			(effects
-				(font
-					(size 1 1)
-					(thickness 0.15)
-				)
-			)
-		)
-		(pad "1" thru_hole circle
-			(at 0 0 90)
-			(size 1.4 1.4)
-			(drill 0.7)
-			(layers "*.Cu" "*.Mask")
-			(remove_unused_layers no)
-		)
-		(pad "1" thru_hole circle
-			(at 2 0 90)
-			(size 1.4 1.4)
-			(drill 0.7)
-			(layers "*.Cu" "*.Mask")
-			(remove_unused_layers no)
-		)
-		(embedded_fonts no)
-		(model "${KICAD9_3DMODEL_DIR}/TestPoint.3dshapes/TestPoint_Bridge_Pitch2.0mm_Drill0.7mm.step"
-			(offset
-				(xyz 0 0 0)
-			)
-			(scale
-				(xyz 1 1 1)
-			)
-			(rotate
-				(xyz 0 0 0)
-			)
 		)
 	)
@@
 		)
 	)
-	(gr_text "DRIVER MOTOR"
-		(at 82 109.3 0)
-		(layer "F.Cu")
-		(effects
-			(font
-				(size 1.5 1.5)
-				(thickness 0.3)
-				(bold yes)
-			)
-			(justify left bottom)
-		)
-	)
-	(gr_text "ALIMENTACIO"
-		(at 112.625 59.475 0)
-		(layer "F.Cu")
-		(effects
-			(font
-				(size 1.5 1.5)
-				(thickness 0.3)
-				(bold yes)
-			)
-			(justify left bottom)
-		)
-	)

Commit message: PCB FIXIng
Other:
- board outline added: 122.8 x 103.7 mm
Changed lines of the file:
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@@
 		)
+	)
+	(gr_rect
+		(start 77.7 53)
+		(end 200.5 156.7)
+		(stroke
+			(width 0.2)
+			(type solid)
+		)
+		(fill no)
+		(layer "Edge.Cuts")
 	)
 	(segment
