File: KiCad/Grup_D_Llums.kicad_pcb (KiCad board)
At the start: 2 copper layers, 122.8 x 103.7 mm, 93 parts, among them J1 DE9_Pins, J2 Screw_Terminal_01x02, J3 Screw_Terminal_01x02, J4 Conn_PIC_ICSP_ICD, J5 DE9_Pins, J6 Screw_Terminal_01x02, J7 Conn_01x10_Pin, Q1 AO3400A, Q2 AO3400A, Q3 AO3400A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

Commit message: Ayuda
Routing:
- net VBAT: track 237.6 -> 238.7 mm
Changed lines of the file:
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@@
 		(layer "Edge.Cuts")
 	)
+	(dimension
+		(type orthogonal)
+		(layer "Edge.Cuts")
+		(pts
+			(xy 200.5 53) (xy 200.5 156.7)
+		)
+		(height 19.5)
+		(orientation 1)
+		(format
+			(prefix "")
+			(suffix "")
+			(units 3)
+			(units_format 0)
+			(precision 4)
+			(suppress_zeroes yes)
+		)
+		(style
+			(thickness 0.05)
+			(arrow_length 1.27)
+			(text_position_mode 0)
+			(arrow_direction outward)
+			(extension_height 0.58642)
+			(extension_offset 0.5)
+			(keep_text_aligned yes)
+		)
+		(gr_text "103,7"
+			(at 218.85 104.85 90)
+			(layer "Edge.Cuts")
+			(effects
+				(font
+					(size 1 1)
+					(thickness 0.15)
+				)
+			)
+		)
+	)
+	(dimension
+		(type orthogonal)
+		(layer "Edge.Cuts")
+		(pts
+			(xy 77.7 53) (xy 200.5 53)
+		)
+		(height -13)
+		(orientation 0)
+		(format
+			(prefix "")
+			(suffix "")
+			(units 3)
+			(units_format 0)
+			(precision 4)
+			(suppress_zeroes yes)
+		)
+		(style
+			(thickness 0.05)
+			(arrow_length 1.27)
+			(text_position_mode 0)
+			(arrow_direction outward)
+			(extension_height 0.58642)
+			(extension_offset 0.5)
+			(keep_text_aligned yes)
+		)
+		(gr_text "122,8"
+			(at 139.1 38.85 0)
+			(layer "Edge.Cuts")
+			(effects
+				(font
+					(size 1 1)
+					(thickness 0.15)
+				)
+			)
+		)
+	)
 	(segment
 		(start 172.8125 57.5125)
@@
 	)
 	(segment
-		(start 149.5385 78.674)
-		(end 148.6125 79.6)
+		(start 119.36 109.9)
+		(end 119.36 104.320818)
 		(width 0.3)
 		(layer "F.Cu")
@@
 	)
 	(segment
-		(start 127.86 71.19)
-		(end 127.845 71.175)
-		(width 0.2)
+		(start 149.5385 78.674)
+		(end 148.6125 79.6)
+		(width 0.3)
 		(layer "F.Cu")
 		(net 12)
@@
 	)
 	(segment
+		(start 150.2 140)
+		(end 184 140)
+		(width 0.3)
+		(layer "F.Cu")
+		(net 12)
+	)
+	(segment
+		(start 127.86 71.19)
+		(end 127.845 71.175)
+		(width 0.2)
+		(layer "F.Cu")
+		(net 12)
+	)
+	(segment
 		(start 149.526 80.5135)
 		(end 148.6125 79.6)
@@
 	)
 	(segment
-		(start 119.36 109.9)
-		(end 119.36 104.320818)
+		(start 184 140)
+		(end 193.5 130.5)
 		(width 0.3)
 		(layer "F.Cu")
@@
 	)
 	(segment
-		(start 182.4 74.8)
-		(end 172.94475 84.25525)
+		(start 120.111818 103.569)
+		(end 124.421 103.569)
 		(width 0.3)
 		(layer "F.Cu")
@@
 	)
 	(segment
-		(start 190.6 74.8)
-		(end 182.4 74.8)
-		(width 0.3)
-		(layer "F.Cu")
-		(net 12)
-	)
-	(segment
 		(start 148.525 58.2)
 		(end 149.5365 59.2115)
@@
 	)
 	(segment
-		(start 185.339 138.661)
-		(end 193.5 130.5)
+		(start 151.89213 87.074)
+		(end 149.526 84.70787)
 		(width 0.3)
 		(layer "F.Cu")
@@
 	)
 	(segment
-		(start 120.111818 103.569)
-		(end 124.421 103.569)
+		(start 149.5385 73.4385)
+		(end 149.5385 78.674)
 		(width 0.3)
 		(layer "F.Cu")
@@
 	)
 	(segment
-		(start 151.89213 87.074)
-		(end 149.526 84.70787)
+		(start 149.526 71.547)
+		(end 148.5865 72.4865)
 		(width 0.3)
 		(layer "F.Cu")
@@
 	)
 	(segment
-		(start 148.861 138.661)
-		(end 185.339 138.661)
+		(start 193.5 77.7)
+		(end 190.6 74.8)
 		(width 0.3)
 		(layer "F.Cu")
@@
 	)
 	(segment
-		(start 149.5385 73.4385)
-		(end 149.5385 78.674)
+		(start 182.4 74.8)
+		(end 172.94475 84.25525)
 		(width 0.3)
 		(layer "F.Cu")
@@
 	)
 	(segment
-		(start 149.526 71.547)
-		(end 148.5865 72.4865)
+		(start 170.126 87.074)
+		(end 151.89213 87.074)
 		(width 0.3)
 		(layer "F.Cu")
@@
 	)
 	(segment
-		(start 138.4 128.2)
-		(end 148.861 138.661)
+		(start 149.5365 59.2115)
+		(end 149.5365 64.1885)
 		(width 0.3)
 		(layer "F.Cu")
@@
 	)
 	(segment
-		(start 170.126 87.074)
-		(end 151.89213 87.074)
+		(start 149.526 84.70787)
+		(end 149.526 80.5135)
 		(width 0.3)
 		(layer "F.Cu")
@@
 	)
 	(segment
-		(start 193.5 77.7)
-		(end 190.6 74.8)
+		(start 148.525 65.2)
+		(end 149.526 66.201)
 		(width 0.3)
 		(layer "F.Cu")
@@
 	)
 	(segment
-		(start 149.5365 59.2115)
-		(end 149.5365 64.1885)
+		(start 190.6 74.8)
+		(end 182.4 74.8)
 		(width 0.3)
 		(layer "F.Cu")
@@
 	)
 	(segment
-		(start 193.5 130.5)
-		(end 193.5 77.7)
+		(start 172.94475 84.25525)
+		(end 170.126 87.074)
 		(width 0.3)
 		(layer "F.Cu")
@@
 	)
 	(segment
-		(start 149.526 84.70787)
-		(end 149.526 80.5135)
-		(width 0.3)
-		(layer "F.Cu")
-		(net 12)
-	)
-	(segment
-		(start 148.525 65.2)
-		(end 149.526 66.201)
+		(start 148.5865 72.4865)
+		(end 149.5385 73.4385)
 		(width 0.3)
 		(layer "F.Cu")
@@
 	)
 	(segment
-		(start 172.94475 84.25525)
-		(end 170.126 87.074)
+		(start 138.4 128.2)
+		(end 150.2 140)
 		(width 0.3)
 		(layer "F.Cu")
@@
 	)
 	(segment
-		(start 148.5865 72.4865)
-		(end 149.5385 73.4385)
+		(start 193.5 130.5)
+		(end 193.5 77.7)
 		(width 0.3)
 		(layer "F.Cu")

Commit message: jeje
Parts:
- moved C11 11.2 mm to (119.3, 95.9), turned to 0 degrees
- moved C1 0.25 mm to (94.7, 89.9)
Routing:
- net VCC: track 135.3 -> 140.7 mm
- net GND: track 142.7 -> 144.5 mm, vias 143 -> 144
Changed lines of the file:
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@@
 	(footprint "Capacitor_SMD:C_0805_2012Metric"
 		(layer "F.Cu")
-		(at 112.125 87.325 180)
+		(at 119.3 95.9)
 		(descr "Capacitor SMD 0805 (2012 Metric), square (rectangular) end terminal, IPC-7351 nominal, (Body size source: IPC-SM-782 page 76, https://www.pcb-3d.com/wordpress/wp-content/uploads/ipc-sm-782a_amendment_1_and_2.pdf, https://docs.google.com/spreadsheets/d/1BsfQQcO9C6DZCsRaXUlFlo91Tg2WpOkGARC1WS5S8t0/edit?usp=sharing), generated with kicad-footprint-generator")
 		(tags "capacitor")
@@
 		(attr smd)
 		(fp_line
-			(start -0.261252 0.735)
-			(end 0.261252 0.735)
+			(start -0.261252 -0.735)
+			(end 0.261252 -0.735)
 			(stroke
 				(width 0.12)
@@
 		)
 		(fp_line
-			(start -0.261252 -0.735)
-			(end 0.261252 -0.735)
+			(start -0.261252 0.735)
+			(end 0.261252 0.735)
 			(stroke
 				(width 0.12)
@@
 		)
 		(pad "1" smd roundrect
-			(at -0.95 0 180)
+			(at -0.95 0)
 			(size 1 1.45)
 			(layers "F.Cu" "F.Mask" "F.Paste")
@@
 		)
 		(pad "2" smd roundrect
-			(at 0.95 0 180)
+			(at 0.95 0)
 			(size 1 1.45)
 			(layers "F.Cu" "F.Mask" "F.Paste")
@@
 	(footprint "Capacitor_THT:CP_Radial_D8.0mm_P3.50mm"
 		(layer "F.Cu")
-		(at 94.527651 89.725 180)
+		(at 94.7 89.9 180)
 		(descr "CP, Radial series, Radial, pin pitch=3.50mm, diameter=8mm, height=12mm, Electrolytic Capacitor")
 		(tags "CP Radial series Radial pin pitch 3.50mm diameter 8mm height 12mm Electrolytic Capacitor")
@@
 	)
 	(segment
+		(start 121.6 95.95)
+		(end 120.3 95.95)
+		(width 0.2)
+		(layer "F.Cu")
+		(net 1)
+	)
+	(segment
 		(start 157.075331 137.485)
 		(end 155.915 137.485)
@@
 	)
 	(segment
+		(start 120.2 97.3)
+		(end 120.25 97.25)
+		(width 0.2)
+		(layer "F.Cu")
+		(net 1)
+	)
+	(segment
 		(start 158.075331 92.024669)
 		(end 158.1 92)
@@
 	)
 	(segment
+		(start 120.25 97.35)
+		(end 120.2 97.3)
+		(width 0.2)
+		(layer "F.Cu")
+		(net 1)
+	)
+	(segment
 		(start 148.6625 84.1)
 		(end 148.6625 82.9625)
@@
 	)
 	(segment
-		(start 111.175 86.075)
-		(end 111.1 86)
-		(width 0.2)
-		(layer "F.Cu")
-		(net 1)
-	)
-	(segment
 		(start 144.015 106.785)
 		(end 144 106.8)
@@
 	)
 	(segment
-		(start 110.125 87.325)
-		(end 110.1 87.3)
-		(width 0.2)
-		(layer "F.Cu")
-		(net 1)
-	)
-	(segment
 		(start 117.5 80.6)
 		(end 117.525 80.575)
@@
 	)
 	(segment
+		(start 120.25 94.45)
+		(end 120.25 95.9)
+		(width 0.2)
+		(layer "F.Cu")
+		(net 1)
+	)
+	(segment
 		(start 172.9 73.7)
 		(end 172.9 72.475)
@@
 	)
 	(segment
+		(start 120.3 95.95)
+		(end 120.25 95.9)
+		(width 0.2)
+		(layer "F.Cu")
+		(net 1)
+	)
+	(segment
 		(start 167.485 108.185)
 		(end 167.5 108.2)
@@
 	)
 	(segment
-		(start 111.175 87.325)
-		(end 110.125 87.325)
-		(width 0.2)
-		(layer "F.Cu")
-		(net 1)
-	)
-	(segment
 		(start 167.4 60.1)
 		(end 167.4 61.3625)
@@
 	)
 	(segment
-		(start 111.175 87.325)
-		(end 111.175 86.075)
-		(width 0.2)
-		(layer "F.Cu")
-		(net 1)
-	)
-	(segment
 		(start 116.375 80.575)
 		(end 116.4 80.6)
@@
 	)
 	(segment
+		(start 120.25 97.25)
+		(end 120.25 95.9)
+		(width 0.2)
+		(layer "F.Cu")
+		(net 1)
+	)
+	(segment
 		(start 153.625331 96.874669)
 		(end 152.7 97.8)
@@
 	)
 	(via
+		(at 121.6 95.95)
+		(size 0.6)
+		(drill 0.3)
+		(layers "F.Cu" "B.Cu")
+		(free yes)
+		(net 1)
+	)
+	(via
 		(at 190 108.9)
 		(size 0.6)
@@
 	)
 	(via
-		(at 111.1 86)
-		(size 0.6)
-		(drill 0.3)
-		(layers "F.Cu" "B.Cu")
-		(free yes)
-		(net 1)
-	)
-	(via
 		(at 153.1 81.60625)
 		(size 0.6)
@@
 	)
 	(via
+		(at 120.25 94.45)
+		(size 0.6)
+		(drill 0.3)
+		(layers "F.Cu" "B.Cu")
+		(free yes)
+		(net 1)
+	)
+	(via
 		(at 113.7 120.9)
 		(size 0.6)
@@
 	)
 	(via
+		(at 120.25 97.35)
+		(size 0.6)
+		(drill 0.3)
+		(layers "F.Cu" "B.Cu")
+		(free yes)
+		(net 1)
+	)
+	(via
 		(at 153.9 61.4)
 		(size 0.6)
@@
 	)
 	(via
-		(at 110.1 87.3)
-		(size 0.6)
-		(drill 0.3)
-		(layers "F.Cu" "B.Cu")
-		(free yes)
-		(net 1)
-	)
-	(via
 		(at 190 102.5)
 		(size 0.6)
@@
 	)
 	(segment
-		(start 103.175 89.825)
-		(end 94.627651 89.825)
-		(width 0.2)
+		(start 102.85 89.9)
+		(end 94.7 89.9)
+		(width 0.5)
 		(layer "F.Cu")
 		(net 2)
 	)
 	(segment
-		(start 110.725 82.275)
-		(end 113.575 82.275)
-		(width 0.2)
+		(start 102.925 89.825)
+		(end 102.85 89.9)
+		(width 0.5)
 		(layer "F.Cu")
 		(net 2)
 	)
 	(segment
-		(start 111.0225 89.825)
-		(end 111.0725 89.775)
-		(width 0.2)
+		(start 94.7 89.9)
+		(end 94.7 84.15)
+		(width 0.5)
 		(layer "F.Cu")
 		(net 2)
@@
 	)
 	(segment
-		(start 94.527651 89.725)
-		(end 94.527651 83.977651)
-		(width 0.2)
+		(start 103.175 89.825)
+		(end 111.0225 89.825)
+		(width 0.5)
 		(layer "F.Cu")
 		(net 2)
 	)
 	(segment
-		(start 103.175 89.825)
-		(end 111.0225 89.825)
-		(width 0.2)
+		(start 111.0225 89.825)
+		(end 111.0725 89.775)
+		(width 0.5)
 		(layer "F.Cu")
 		(net 2)
 	)
 	(segment
-		(start 103.175 89.825)
+		(start 110.725 82.275)
+		(end 103.175 89.825)
+		(width 0.5)
+		(layer "F.Cu")
+		(net 2)
+	)
+	(segment
+		(start 113.575 82.275)
 		(end 110.725 82.275)
-		(width 0.2)
+		(width 0.5)
+		(layer "F.Cu")
+		(net 2)
+	)
+	(segment
+		(start 103.175 89.825)
+		(end 102.925 89.825)
+		(width 0.5)
+		(layer "F.Cu")
+		(net 2)
+	)
+	(segment
+		(start 94.7 84.15)
+		(end 94.375 83.825)
+		(width 0.5)
 		(layer "F.Cu")
 		(net 2)
@@
 	)
 	(segment
+		(start 113.075 89.4975)
+		(end 113.3525 89.775)
+		(width 0.2)
+		(layer "F.Cu")
+		(net 5)
+	)
+	(segment
 		(start 154.925331 96.585)
 		(end 154.925331 99.385)
@@
 	)
 	(segment
+		(start 118.35 95.9)
+		(end 113.5275 95.9)
+		(width 0.2)
+		(layer "F.Cu")
+		(net 5)
+	)
+	(segment
 		(start 151.350331 114.685)
 		(end 150.250331 113.585)
@@
 		(width 0.2)
 		(layer "F.Cu")
+		(net 5)
+	)
+	(segment
+		(start 113.5275 95.9)
+		(end 113.3525 96.075)
+		(width 0.2)
+		(layer "F.Cu")

Commit message: hotfix
Connections:
- net Net-(D1-K) renamed OUTLM
- net Net-(D3-K) renamed VIN
Routing:
- net VCC: track 140.7 -> 125.4 mm
- net GND: track 144.5 -> 145.7 mm
