File: KiCad/Grup_D_Llums.kicad_pcb (KiCad board)
At the start: 2 copper layers, 122.8 x 103.7 mm, 93 parts, among them J1 DE9_Pins, J2 Screw_Terminal_01x02, J3 Screw_Terminal_01x02, J4 Conn_PIC_ICSP_ICD, J5 DE9_Pins, J6 Screw_Terminal_01x02, J7 Conn_01x10_Pin, Q1 AO3400A, Q2 AO3400A, Q3 AO3400A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

Commit message: A
Parts:
- removed F1, F2, F3, F4, F5, F6, F7, F8: Fuse, Fuse:Fuse_0805_2012Metric
- removed REF** (x4): MountingHole_2.2mm_M2, MountingHole:MountingHole_2.2mm_M2
- added J10: Screw_Terminal_01x02, TerminalBlock_Phoenix:TerminalBlock_Phoenix_MKDS-1,5-2-5.08_1x02_P5.08mm_Horizontal, F.Cu at (80.1, 85.9)
- added J11: Screw_Terminal_01x02, TerminalBlock_Phoenix:TerminalBlock_Phoenix_MKDS-1,5-2-5.08_1x02_P5.08mm_Horizontal, F.Cu at (92.3, 73.8)
- added J12: Screw_Terminal_01x02, TerminalBlock_Phoenix:TerminalBlock_Phoenix_MKDS-1,5-2-5.08_1x02_P5.08mm_Horizontal, F.Cu at (92.3, 85.9)
- added J13: Screw_Terminal_01x02, TerminalBlock_Phoenix:TerminalBlock_Phoenix_MKDS-1,5-2-5.08_1x02_P5.08mm_Horizontal, F.Cu at (104.5, 73.8)
- added J14: Screw_Terminal_01x02, TerminalBlock_Phoenix:TerminalBlock_Phoenix_MKDS-1,5-2-5.08_1x02_P5.08mm_Horizontal, F.Cu at (104.5, 85.9)
- added J8: Screw_Terminal_01x02, TerminalBlock_Phoenix:TerminalBlock_Phoenix_MKDS-1,5-2-5.08_1x02_P5.08mm_Horizontal, F.Cu at (67.9, 85.9)
- added J9: Screw_Terminal_01x02, TerminalBlock_Phoenix:TerminalBlock_Phoenix_MKDS-1,5-2-5.08_1x02_P5.08mm_Horizontal, F.Cu at (80.1, 73.8)
- J7: value Conn_01x10_Pin -> Screw_Terminal_01x02; footprint Connector_PinHeader_2.54mm:PinHeader_1x10_P2.54mm_Vertical -> TerminalBlock_Phoenix:TerminalBlock_Phoenix_MKDS-1,5-2-5.08_1x02_P5.08mm_Horizontal
- moved J2 137.7 mm to (32.7, 146.0), turned to 0 degrees
- moved D7 136.9 mm to (20.7, 53.7), turned to 0 degrees
- moved D8 136.3 mm to (20.7, 60.5), turned to 0 degrees
- moved J1 133.7 mm to (97.3, 18.9), turned to 0 degrees
- moved SW2 130.5 mm to (69.8, 21.6), turned to 0 degrees
- moved J6 128.5 mm to (41.9, 47.1)
- moved SW4 128.5 mm to (69.8, 41.2)
- moved SW7 127.8 mm to (52.6, 30.1), turned to 0 degrees
- moved SW3 126.9 mm to (69.8, 31.4), turned to 0 degrees
- moved D5 120.9 mm to (20.7, 40.2)
- moved SW5 118.4 mm to (69.8, 51.0), turned to 0 degrees
- moved C7 113.7 mm to (114.9, 35.4)
- moved C6 113.5 mm to (114.9, 32.4), turned to 0 degrees
- moved D6 111.3 mm to (20.7, 47.0)
- moved C3 110.8 mm to (110.5, 35.4)
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Connections:
- D6 pad 1: VCC -> GND
- D6 pad 2: Net-(D11-A) -> Net-(D5-A)
- D7 pad 2: Net-(D10-A) -> Net-(D11-A)
- D9 pad 1: GND -> VCC
- D9 pad 2: Net-(D5-A) -> Net-(D10-A)
- J7 pad 1: unconnected-(J7-Pin_1-Pad1) -> VBAT
- J7 pad 2: LOW_R -> DRL_O
- Q1 pad 1: Net-(Q1-G) -> VBAT
- Q2 pad 1: Net-(Q2-G) -> VBAT
- Q3 pad 1: Net-(Q3-G) -> VBAT
- Q4 pad 1: Net-(Q4-G) -> VBAT
- Q5 pad 1: Net-(Q5-G) -> VBAT
- Q6 pad 1: Net-(Q6-G) -> VBAT
- Q7 pad 1: Net-(Q7-G) -> VBAT
- Q8 pad 1: Net-(Q8-G) -> VBAT
- R1 pad 1: Net-(Q1-G) -> VBAT
- R10 pad 1: Net-(Q5-G) -> VBAT
- R15 pad 2: Net-(Q6-G) -> VBAT
- R16 pad 1: Net-(Q6-G) -> VBAT
- R17 pad 2: Net-(Q7-G) -> VBAT
- R18 pad 1: Net-(Q7-G) -> VBAT
- R19 pad 2: Net-(Q8-G) -> VBAT
- R2 pad 2: Net-(Q1-G) -> VBAT
- R20 pad 1: Net-(Q8-G) -> VBAT
- R3 pad 2: Net-(Q2-G) -> VBAT
- R4 pad 1: Net-(Q2-G) -> VBAT
- R5 pad 2: Net-(Q3-G) -> VBAT
- R6 pad 1: Net-(Q3-G) -> VBAT
- R7 pad 2: Net-(Q4-G) -> VBAT
- R8 pad 1: Net-(Q4-G) -> VBAT
- R9 pad 2: Net-(Q5-G) -> VBAT
- U1 pad 12: LF_FWD -> LF_PWM
- U1 pad 8: LF_PWM -> LF_FWD
Routing:
- net VBAT: track 238.7 -> 6.13 mm
- net GND: track 145.7 -> 0.00 mm, vias 144 -> 0
- net Net-(D11-A): track 132.5 -> 0.00 mm
- net VCC: track 125.4 -> 8.97 mm
- net HI_BEAM_CTRL: track 106.9 -> 0.00 mm
- net LOW_BEAM_CTRL: track 88.9 -> 0.00 mm
- net Net-(D10-A): track 69.4 -> 0.00 mm
- net Net-(D12-A): track 64.9 -> 0.00 mm
- net LF_FWD: track 47.5 -> 0.00 mm
- net LF_REV: track 47.5 -> 0.00 mm
- net TURN_RIGHT_CTRL: track 46.2 -> 0.00 mm
- net LF_PWM: track 45.2 -> 0.00 mm
- net TURN_LEFT_CTRL: track 38.2 -> 0.00 mm
- net Net-(D5-A): track 37.2 -> 0.00 mm
- net Usart1: track 35.2 -> 0.00 mm
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- removed copper zone on B.Cu, net GND
- removed copper zone on F.Cu, net GND
- removed copper zone on F.Cu, net VBAT
- removed copper zone on F.Cu, net VCC
Other:
- board outline removed

Commit message: a
Parts:
- moved C1 130.8 mm to (206.1, 110.0)
- moved C10 130.8 mm to (201.2, 119.0)
- moved C11 130.8 mm to (202.7, 99.8)
- moved C9 130.8 mm to (182.6, 103.3)
- moved D1 130.8 mm to (191.5, 127.5)
- moved D3 130.8 mm to (185.0, 110.3)
- moved D4 130.8 mm to (185.1, 118.8)
- moved J2 130.8 mm to (158.6, 110.3)
- moved L1 130.8 mm to (191.3, 118.9)
- moved U2 130.8 mm to (193.7, 102.8)
- moved U7 130.8 mm to (211.3, 99.8)
Changed lines of the file:
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@@
 	(footprint "Capacitor_SMD:C_0805_2012Metric"
 		(layer "F.Cu")
-		(at 76.8 135.45 180)
+		(at 202.65 99.8 180)
 		(descr "Capacitor SMD 0805 (2012 Metric), square (rectangular) end terminal, IPC-7351 nominal, (Body size source: IPC-SM-782 page 76, https://www.pcb-3d.com/wordpress/wp-content/uploads/ipc-sm-782a_amendment_1_and_2.pdf, https://docs.google.com/spreadsheets/d/1BsfQQcO9C6DZCsRaXUlFlo91Tg2WpOkGARC1WS5S8t0/edit?usp=sharing), generated with kicad-footprint-generator")
 		(tags "capacitor")
@@
 	(footprint "Inductor_THT:L_Radial_D10.0mm_P5.00mm_Fastron_07M"
 		(layer "F.Cu")
-		(at 65.5 154.55)
+		(at 191.35 118.9)
 		(descr "Inductor, Radial series, Radial, pin pitch=5.00mm, diameter=10mm, height=12.7mm, Fastron, 07M, http://www.fastrongroup.com/image-show/37/07M.pdf?type=Complete-DataSheet&productType=series")
 		(tags "Inductor Radial series Radial pin pitch 5.00mm  diameter 10mm height 12.7mm Fastron 07M")
@@
 	(footprint "Capacitor_THT:CP_Radial_D10.0mm_P5.00mm"
 		(layer "F.Cu")
-		(at 56.7 139 90)
+		(at 182.55 103.35 90)
 		(descr "CP, Radial series, Radial, pin pitch=5.00mm, diameter=10mm, height=16mm, Electrolytic Capacitor")
 		(tags "CP Radial series Radial pin pitch 5.00mm diameter 10mm height 16mm Electrolytic Capacitor")
@@
 	(footprint "Diode_THT:D_DO-201AD_P15.24mm_Horizontal"
 		(layer "F.Cu")
-		(at 59.17 146 180)
+		(at 185.02 110.35 180)
 		(descr "Diode, DO-201AD series, Axial, Horizontal, pin pitch=15.24mm, length*diameter=9.5*5.2mm^2, http://www.diodes.com/_files/packages/DO-201AD.pdf")
 		(tags "Diode DO-201AD series Axial Horizontal pin pitch 15.24mm  length 9.5mm diameter 5.2mm")
@@
 	(footprint "Package_TO_SOT_SMD:TO-252-3_TabPin2"
 		(layer "F.Cu")
-		(at 85.44 135.5)
+		(at 211.29 99.85)
 		(descr "TO-252/DPAK SMD package, http://www.infineon.com/cms/en/product/packages/PG-TO252/PG-TO252-3-1/")
 		(tags "DPAK TO-252 DPAK-3 TO-252-3 SOT-428")
@@
 	(footprint "TerminalBlock_Phoenix:TerminalBlock_Phoenix_MKDS-1,5-2-5.08_1x02_P5.08mm_Horizontal"
 		(layer "F.Cu")
-		(at 32.72 146)
+		(at 158.57 110.35)
 		(descr "Terminal Block Phoenix MKDS-1,5-2-5.08, 2 pins, pitch 5.08mm, size 10.2x9.8mm, drill diameter 1.3mm, pad diameter 2.6mm, http://www.farnell.com/datasheets/100425.pdf, script-generated using https://gitlab.com/kicad/libraries/kicad-footprint-generator/-/tree/master/scripts/TerminalBlock_Phoenix")
 		(tags "THT Terminal Block Phoenix MKDS-1,5-2-5.08 pitch 5.08mm size 10.2x9.8mm drill 1.3mm pad 2.6mm")
@@
 	(footprint "Package_TO_SOT_SMD:TO-263-5_TabPin3"
 		(layer "F.Cu")
-		(at 67.85 138.45 90)
+		(at 193.7 102.8 90)
 		(descr "TO-263/D2PAK/DDPAK SMD package, http://www.infineon.com/cms/en/product/packages/PG-TO263/PG-TO263-5-1/")
 		(tags "D2PAK DDPAK TO-263 D2PAK-5 TO-263-5 SOT-426")
@@
 	(footprint "Capacitor_SMD:C_0805_2012Metric"
 		(layer "F.Cu")
-		(at 75.3 154.7)
+		(at 201.15 119.05)
 		(descr "Capacitor SMD 0805 (2012 Metric), square (rectangular) end terminal, IPC-7351 nominal, (Body size source: IPC-SM-782 page 76, https://www.pcb-3d.com/wordpress/wp-content/uploads/ipc-sm-782a_amendment_1_and_2.pdf, https://docs.google.com/spreadsheets/d/1BsfQQcO9C6DZCsRaXUlFlo91Tg2WpOkGARC1WS5S8t0/edit?usp=sharing), generated with kicad-footprint-generator")
 		(tags "capacitor")
@@
 	(footprint "Capacitor_THT:CP_Radial_D8.0mm_P3.50mm"
 		(layer "F.Cu")
-		(at 80.2 145.65)
+		(at 206.05 110)
 		(descr "CP, Radial series, Radial, pin pitch=3.50mm, diameter=8mm, height=12mm, Electrolytic Capacitor")
 		(tags "CP Radial series Radial pin pitch 3.50mm diameter 8mm height 12mm Electrolytic Capacitor")
@@
 	(footprint "Diode_THT:D_DO-201AD_P15.24mm_Horizontal"
 		(layer "F.Cu")
-		(at 59.27 154.4 180)
+		(at 185.12 118.75 180)
 		(descr "Diode, DO-201AD series, Axial, Horizontal, pin pitch=15.24mm, length*diameter=9.5*5.2mm^2, http://www.diodes.com/_files/packages/DO-201AD.pdf")
 		(tags "Diode DO-201AD series Axial Horizontal pin pitch 15.24mm  length 9.5mm diameter 5.2mm")
@@
 	(footprint "Diode_THT:D_DO-201AD_P15.24mm_Horizontal"
 		(layer "F.Cu")
-		(at 65.68 163.1)
+		(at 191.53 127.45)
 		(descr "Diode, DO-201AD series, Axial, Horizontal, pin pitch=15.24mm, length*diameter=9.5*5.2mm^2, http://www.diodes.com/_files/packages/DO-201AD.pdf")
 		(tags "Diode DO-201AD series Axial Horizontal pin pitch 15.24mm  length 9.5mm diameter 5.2mm")
@@
 		)
 	)
+	(gr_rect
+		(start 150.4 50.95)
+		(end 252.4 129.8)
+		(stroke
+			(width 0.2)
+			(type default)
+		)
+		(fill no)
+		(layer "F.Cu")
+		(net 10)
+	)
 	(segment
-		(start 69.55 153.6)
-		(end 69.55 146.1)
+		(start 195.4 117.95)
+		(end 195.4 110.45)
 		(width 0.5)
 		(layer "F.Cu")
@@
 	)
 	(segment
-		(start 80.4 137.78)
-		(end 80.4 145.45)
+		(start 206.25 102.13)
+		(end 206.25 109.8)
 		(width 0.5)
 		(layer "F.Cu")
@@
 	)
 	(segment
-		(start 74.35 151.5)
-		(end 80.2 145.65)
+		(start 200.2 115.85)
+		(end 206.05 110)
 		(width 0.5)
 		(layer "F.Cu")
@@
 	)
 	(segment
-		(start 74.35 154.7)
-		(end 74.35 151.5)
+		(start 200.2 119.05)
+		(end 200.2 115.85)
 		(width 0.5)
 		(layer "F.Cu")
@@
 	)
 	(segment
-		(start 80.4 145.45)
-		(end 80.2 145.65)
+		(start 206.25 109.8)
+		(end 206.05 110)
 		(width 0.5)
 		(layer "F.Cu")
@@
 	)
 	(segment
-		(start 70.5 154.55)
-		(end 69.55 153.6)
+		(start 196.35 118.9)
+		(end 195.4 117.95)
 		(width 0.5)
 		(layer "F.Cu")
@@
 	)
 	(segment
-		(start 74.2 154.55)
-		(end 74.35 154.7)
+		(start 200.05 118.9)
+		(end 200.2 119.05)
 		(width 0.5)
 		(layer "F.Cu")
@@
 	)
 	(segment
-		(start 70.5 154.55)
-		(end 74.2 154.55)
+		(start 196.35 118.9)
+		(end 200.05 118.9)
 		(width 0.5)
 		(layer "F.Cu")
@@
 	)
 	(segment
-		(start 80.4 135.5)
-		(end 86.7 135.5)
+		(start 206.25 99.85)
+		(end 212.55 99.85)
 		(width 0.2)
 		(layer "F.Cu")
@@
 	)
 	(segment
-		(start 80.4 135.5)
-		(end 77.8 135.5)
+		(start 206.25 99.85)
+		(end 203.65 99.85)
 		(width 0.2)
 		(layer "F.Cu")
@@
 	)
 	(segment
-		(start 77.8 135.5)
-		(end 77.75 135.45)
+		(start 203.65 99.85)
+		(end 203.6 99.8)
 		(width 0.2)
 		(layer "F.Cu")
@@
 	)
 	(segment
-		(start 37.8 146)
-		(end 43.93 146)
+		(start 163.65 110.35)
+		(end 169.78 110.35)
 		(width 0.8)
 		(layer "F.Cu")
@@
 	)
 	(segment
-		(start 59.17 141.47)
-		(end 56.7 139)
+		(start 185.02 105.82)
+		(end 182.55 103.35)
 		(width 0.8)
 		(layer "F.Cu")
@@
 	)
 	(segment
-		(start 59.17 146)
-		(end 64.35 146)
+		(start 185.02 110.35)
+		(end 190.2 110.35)
 		(width 0.8)
 		(layer "F.Cu")
@@
 	)
 	(segment
-		(start 59.27 146.1)
-		(end 59.17 146)
+		(start 185.12 110.45)
+		(end 185.02 110.35)
 		(width 0.8)
 		(layer "F.Cu")
@@
 	)
 	(segment
-		(start 59.17 146)
-		(end 59.17 141.47)
+		(start 185.02 110.35)
+		(end 185.02 105.82)
 		(width 0.8)
 		(layer "F.Cu")
@@
 	)
 	(segment
-		(start 59.27 154.4)
-		(end 59.27 146.1)
+		(start 185.12 118.75)
+		(end 185.12 110.45)
 		(width 0.8)
 		(layer "F.Cu")
@@
 	)
 	(segment
-		(start 64.35 146)
-		(end 64.45 146.1)
+		(start 190.2 110.35)
+		(end 190.3 110.45)
 		(width 0.8)
 		(layer "F.Cu")
@@
 	)
 	(segment
-		(start 66.15 146.1)
-		(end 66.1 146.15)
+		(start 192 110.45)
+		(end 191.95 110.5)
 		(width 0.2)
 		(layer "F.Cu")
@@
 	)
 	(segment
-		(start 66.15 146.1)
-		(end 66.15 153.9)
+		(start 192 110.45)
+		(end 192 118.25)
 		(width 0.5)
 		(layer "F.Cu")
@@
 	)
 	(segment
-		(start 66.1 146.15)
-		(end 66.1 146.9)
+		(start 191.95 110.5)
+		(end 191.95 111.25)
 		(width 0.2)
 		(layer "F.Cu")
@@
 	)
 	(segment
-		(start 65.5 162.92)
-		(end 65.68 163.1)
+		(start 191.35 127.27)
+		(end 191.53 127.45)
 		(width 0.2)
 		(layer "F.Cu")
@@
 	)
 	(segment
-		(start 65.5 154.55)
-		(end 65.5 162.92)
+		(start 191.35 118.9)
+		(end 191.35 127.27)
 		(width 0.5)
 		(layer "F.Cu")
@@
 	)
 	(segment
-		(start 66.15 153.9)
-		(end 65.5 154.55)
+		(start 192 118.25)
+		(end 191.35 118.9)
 		(width 0.5)
 		(layer "F.Cu")

Commit message: a
Parts:
- moved C16 138.4 mm to (-52.6, 80.0)
- moved C6 138.4 mm to (-21.7, 10.2)
- moved C7 138.4 mm to (-21.7, 13.2)
- moved C8 138.4 mm to (-21.7, 16.2)
- moved D2 138.4 mm to (-52.4, 40.1)
- moved J4 138.4 mm to (-21.6, 26.7)
- moved Q7 138.4 mm to (-41.9, 71.8)
- moved Q8 138.4 mm to (-41.9, 76.2)
- moved R11 138.4 mm to (-26.1, 25.9)
- moved R12 138.4 mm to (-26.1, 28.8)
- moved R13 138.4 mm to (-26.1, 31.8)
- moved R14 138.4 mm to (-26.1, 34.7)
- moved R19 138.4 mm to (-61.3, 71.0)
- moved R20 138.4 mm to (-61.3, 74.0)
- moved SW2 138.4 mm to (-66.8, -0.66)
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Connections:
- D10 pad 1: GND -> Net-(D10-K)
- D10 pad 2: Net-(D10-A) -> GND
- D11 pad 1: GND -> Net-(D11-K)
- D11 pad 2: Net-(D11-A) -> GND
- D12 pad 1: GND -> Net-(D12-K)
- D12 pad 2: Net-(D12-A) -> GND
- D5 pad 2: Net-(D5-A) -> Net-(D12-K)
- D6 pad 1: GND -> Net-(D6-K)
- D6 pad 2: Net-(D5-A) -> GND
- D7 pad 2: Net-(D11-A) -> Net-(D11-K)
- D8 pad 2: Net-(D10-A) -> Net-(D10-K)
- D9 pad 2: Net-(D10-A) -> Net-(D6-K)
- J3 pad 1: Net-(D5-A) -> Net-(D12-K)
- J3 pad 2: Net-(D11-A) -> Net-(D11-K)
- J6 pad 1: Net-(D10-A) -> Net-(D10-K)
- J6 pad 2: Net-(D12-A) -> Net-(D6-K)
- U3 pad 13: Net-(D10-A) -> Net-(D10-K)
- U3 pad 14: Net-(D12-A) -> Net-(D6-K)
- U3 pad 2: Net-(D5-A) -> Net-(D12-K)
- U3 pad 3: Net-(D11-A) -> Net-(D11-K)
Routing:
- net Net-(D11-K): track 0.00 -> 67.2 mm
- net VBAT: track 6.13 -> 70.3 mm
- net Net-(D6-K): track 0.00 -> 32.9 mm
- net Net-(D10-K): track 0.00 -> 30.7 mm
- net Net-(D12-K): track 0.00 -> 26.2 mm
- net LF_PWM: track 0.00 -> 8.45 mm
- net LF_REV: track 0.00 -> 8.45 mm
- net LF_FWD: track 0.00 -> 8.45 mm
- net VCC: track 8.97 -> 11.7 mm
- added copper zone on F.Cu, net VCC

Commit message: fin1
Parts:
- added REF**: MountingHole_2.1mm, MountingHole:MountingHole_2.1mm, F.Cu at (50.2, 46.1)
- added REF**: MountingHole_2.1mm, MountingHole:MountingHole_2.1mm, F.Cu at (223.2, 142.3)
- added REF**: MountingHole_2.1mm, MountingHole:MountingHole_2.1mm, F.Cu at (222.8, 46.1)
- added REF**: MountingHole_2.1mm, MountingHole:MountingHole_2.1mm, F.Cu at (50.4, 141.1)
- moved SW4 271.0 mm to (195.0, 89.0), turned to 90 degrees
- moved J11 269.1 mm to (211.0, 136.7)
- moved SW2 268.4 mm to (195.0, 58.6), turned to 90 degrees
- moved SW5 266.6 mm to (195.0, 78.9), turned to 90 degrees
- moved SW3 264.8 mm to (195.0, 48.5), turned to 90 degrees
- moved SW6 263.5 mm to (195.0, 68.8), turned to 90 degrees
- moved Q7 263.1 mm to (215.2, 128.0)
- moved Q4 259.3 mm to (202.3, 128.0)
- moved J12 253.2 mm to (198.2, 136.6)
- moved SW7 246.3 mm to (145.3, 97.7), turned to 180 degrees
- moved R8 242.3 mm to (171.2, 121.5)
- moved Q8 236.2 mm to (188.6, 128.1)
- moved R18 231.8 mm to (163.8, 121.5)
- moved pull_FC1 231.2 mm to (149.4, 93.2), turned to 180 degrees
- moved Q5 229.3 mm to (175.5, 128.0)
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Connections:
- net Net-(C3-Pad2) renamed M
- net Net-(D2-K) renamed LedA
- net Net-(U1-RA8) renamed Usart
- net Net-(U1-VBUS) renamed Vbus
- net Net-(U1-VCAP) renamed Vcap
- net Net-(U6-CANH) renamed CanH
- net Net-(U6-CANL) renamed CanL
- U1 pad 12: LF_PWM -> LF_LIMIT
- U1 pad 13: unconnected-(U1-RA7-Pad13) -> IN_CA
- U1 pad 14: unconnected-(U1-RB14-Pad14) -> IN_CR
- U1 pad 23: TXD -> RXD
- U1 pad 24: RXD -> TXD
- U1 pad 26: IN_CA -> unconnected-(U1-RC1-Pad26)
- U1 pad 27: IN_CR -> unconnected-(U1-RC2-Pad27)
- U1 pad 34: LF_LIMIT -> unconnected-(U1-RA4-Pad34)
- U1 pad 35: unconnected-(U1-RA9-Pad35) -> LF_PWM
- U1 pad 36: unconnected-(U1-RC3-Pad36) -> LF_REV
- U1 pad 37: unconnected-(U1-RC4-Pad37) -> LF_FWD
- U1 pad 38: SCL -> unconnected-(U1-RC5-Pad38)
- U1 pad 41: unconnected-(U1-RB5-Pad41) -> SCL
- U1 pad 8: LF_FWD -> unconnected-(U1-RB10-Pad8)
- U1 pad 9: LF_REV -> unconnected-(U1-RB11-Pad9)
Routing:
- net IN_R: track 0.00 -> 77.4 mm
- net IN_L: track 0.00 -> 73.5 mm
- net IN_LF: track 0.00 -> 72.5 mm
- net IN_CR: track 0.00 -> 68.7 mm
- net IN_CA: track 0.00 -> 66.7 mm
- net HI_BEAM_CTRL: track 0.00 -> 39.8 mm
- net LOW_BEAM_CTRL: track 0.00 -> 37.7 mm
- net MCLR: track 0.00 -> 37.4 mm
- net DRL_CTRL: track 0.00 -> 34.8 mm
- net TURN_RIGHT_CTRL: track 0.00 -> 34.1 mm
- net LF_PWM: track 8.45 -> 42.1 mm
- net LF_FWD: track 8.45 -> 42.0 mm
- net TURN_LEFT_CTRL: track 0.00 -> 33.3 mm
- net LF_REV: track 8.45 -> 41.3 mm
- net LF_LIMIT: track 0.00 -> 25.5 mm
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- added copper zone on B.Cu, net GND
- added copper zone on F.Cu, net GND
- added copper zone on F.Cu, net VBAT
Other:
- board outline added: 181.8 x 103.2 mm

Commit message: a
Parts:
- R12, R13: footprint Resistor_SMD:R_0805_2012Metric -> Resistor_SMD:R_0603_1608Metric
- moved Q7 39.1 mm to (182.5, 106.5), turned to 90 degrees
- moved REF** 35.9 mm to (187.4, 142.7)
- moved REF** 35.8 mm to (187.1, 45.7)
- moved J11 32.7 mm to (191.2, 110.6), turned to 90 degrees
- moved Q4 21.6 mm to (182.5, 119.3), turned to 90 degrees
- moved C3 17.2 mm to (133.9, 55.8), turned to -90 degrees
- moved R13 14.9 mm to (134.6, 59.0), turned to -90 degrees
- moved J12 14.9 mm to (191.2, 123.4), turned to 90 degrees
- moved R12 14.6 mm to (133.0, 59.0), turned to 90 degrees
- moved pull_INT1 10.8 mm to (115.3, 89.7)
- moved U9 10.0 mm to (108.7, 89.7), turned to 0 degrees
- moved C16 9.26 mm to (104.9, 89.2)
- moved pull_SCL2 9.20 mm to (107.8, 86.0)
- moved Q8 7.77 mm to (182.6, 133.0), turned to 90 degrees
- moved pull_SDA2 7.15 mm to (111.9, 89.1)
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Routing:
- net VCC: track 23.7 -> 14.5 mm
- net CanH: track 15.1 -> 23.7 mm
- net SCL: track 12.7 -> 19.1 mm
- net TXD: track 13.5 -> 7.78 mm
- net GND: track 5.71 -> 0.21 mm, vias 100 -> 138
- net CanL: track 19.3 -> 15.0 mm
- net M: track 7.27 -> 3.51 mm
- net SDA: track 9.76 -> 13.2 mm
- net Net-(D11-K): track 67.2 -> 68.8 mm
- net RXD: track 11.0 -> 12.5 mm
- net LIGHT_INT: track 13.8 -> 14.4 mm
Other:
- board text added: "C2"

Commit message: a
Parts:
- moved C8 4.22 mm to (126.9, 86.8)
- moved C13 0.97 mm to (124.7, 86.8), turned to 90 degrees
Connections:
- net Net-(D10-K) renamed OUTM3
- net Net-(D11-K) renamed OUTM2
- net Net-(D12-K) renamed OUTM1
- net Net-(D6-K) renamed OUTM4
Routing:
- net 5VOLTS: track 32.2 -> 1.84 mm
- net VIN: track 21.8 -> 0.28 mm
- net GND: track 0.21 -> 19.9 mm, vias 138 -> 174
- net OUTLM: track 18.2 -> 1.74 mm
- net Vcap: track 3.64 -> 2.96 mm
- added copper zone on F.Cu, net 5VOLTS
- added copper zone on F.Cu, net OUTLM
- added copper zone on F.Cu, net VIN

Commit message: a
Other:
- board size 181.8 x 103.2 mm -> 155.3 x 103.2 mm
Changed lines of the file:
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@@
 	(gr_rect
 		(start 45.9 42.6)
-		(end 227.7 145.75)
+		(end 201.2 145.75)
 		(stroke
 			(width 0.05)
@@
 		(polygon
 			(pts
-				(xy 45.9 42.6) (xy 196.8 42.6) (xy 196.8 145.75) (xy 45.9 145.75)
+				(xy 45.9 42.6) (xy 201.13 43.1) (xy 201.13 146.25) (xy 45.9 145.75)
 			)
 		)
@@
 		(polygon
 			(pts
-				(xy 45.85 112.8) (xy 177.3 112.8) (xy 177.3 101.1) (xy 196.8 101.1) (xy 196.8 145.75) (xy 45.9 145.75)
+				(xy 45.85 112.8) (xy 177.3 112.8) (xy 177.3 101.1) (xy 200.76 101.3) (xy 200.76 145.95) (xy 45.9 145.75)
 			)
 		)
@@
 		(polygon
 			(pts
-				(xy 45.9 42.6) (xy 196.8 42.6) (xy 196.8 145.75) (xy 45.9 145.75)
+				(xy 45.9 42.6) (xy 200.99 43.26) (xy 200.99 146.41) (xy 45.9 145.75)
 			)
 		)

Commit message: a
Parts:
- added REF**: TestPoint_Bridge_Pitch2.0mm_Drill0.7mm, TestPoint:TestPoint_Bridge_Pitch2.0mm_Drill0.7mm, F.Cu at (108.7, 81.2)
- added REF**: TestPoint_Bridge_Pitch2.0mm_Drill0.7mm, TestPoint:TestPoint_Bridge_Pitch2.0mm_Drill0.7mm, F.Cu at (112.0, 84.9)
