File: KiCad/Transceptor_CAN.kicad_sch (KiCad schematic)
At the start: 22 parts, among them J1 DE9_Pins, J4 Conn_PIC_ICSP_ICD, J5 DE9_Pins, SW2 SW_SPDT, SW3 SW_SPDT, SW4 SW_SPDT, SW5 SW_SPDT, SW6 SW_SPDT, U1 PIC32MX250F128D-IPT, U6 SN65HVD232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

Commit message: Aa
Parts:
- added D2: LED, symbol Device:LED
- added R11: 1k, symbol Device:R_US
Connections:
- net GND: now also R11.2
- net VCC: now also D2.2 (A)
- new net: D2.1 (K), R11.1
Other:
- note added: "LED ALIMENTACIO"

Commit message: Huellass
Parts:
- C13, C2, C3, C5, C6, C7, C8: footprint (none) -> Capacitor_SMD:C_0805_2012Metric
- D2: footprint (none) -> LED_SMD:LED_0805_2012Metric
- J1, J5: footprint (none) -> Connector_Dsub:DSUB-9_Socket_Horizontal_P2.77x2.84mm_EdgePinOffset9.40mm
- R11, R12, R13: footprint (none) -> Resistor_SMD:R_0805_2012Metric
- SW3, SW4, SW5, SW6: footprint (none) -> Button_Switch_SMD:SW_SPDT_CK_JS102011SAQN
Connections:
- no-connect marks 13 -> 21
Changed lines of the file:
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@@
 	)
 	(no_connect
+		(at 33.02 58.42)
+	)
+	(no_connect
 		(at 142.24 58.42)
 	)
 	(no_connect
+		(at 33.02 83.82)
+	)
+	(no_connect
 		(at 36.83 144.78)
 	)
 	(no_connect
+		(at 73.66 73.66)
+	)
+	(no_connect
 		(at 142.24 63.5)
 	)
@@
 	)
 	(no_connect
+		(at 73.66 55.88)
+	)
+	(no_connect
+		(at 33.02 55.88)
+	)
+	(no_connect
 		(at 36.83 152.4)
 	)
 	(no_connect
+		(at 73.66 86.36)
+	)
+	(no_connect
+		(at 33.02 63.5)
+	)
+	(no_connect
 		(at 142.24 53.34)
 	)
@@
 	)
 	(no_connect
+		(at 33.02 81.28)
+	)
+	(no_connect
 		(at 140.97 153.67)
 	)
@@
 		)
 	)
+	(wire
+		(pts
+			(xy 135.89 137.16) (xy 135.89 135.89)
+		)
+		(stroke
+			(width 0)
+			(type default)
+		)
+	)
 	(polyline
 		(pts
@@
 	)
 	(global_label "TXD"
-		(shape output)
+		(shape input)
 		(at 31.75 50.8 180)
 		(fields_autoplaced yes)
@@
 			)
 		)
-		(property "Footprint" ""
+		(property "Footprint" "LED_SMD:LED_0805_2012Metric"
 			(at 120.65 40.64 0)
 			(effects
@@
 	(symbol
 		(lib_id "power:GND")
-		(at 135.89 135.89 0)
+		(at 135.89 137.16 0)
 		(unit 1)
 		(exclude_from_sim no)
@@
 		(fields_autoplaced yes)
 		(property "Reference" "#PWR01"
-			(at 135.89 142.24 0)
+			(at 135.89 143.51 0)
 			(effects
 				(font
@@
 		)
 		(property "Value" "GND"
-			(at 135.89 140.97 0)
+			(at 135.89 142.24 0)
 			(effects
 				(font
@@
 		)
 		(property "Footprint" ""
-			(at 135.89 135.89 0)
+			(at 135.89 137.16 0)
 			(effects
 				(font
@@
 		)
 		(property "Datasheet" ""
-			(at 135.89 135.89 0)
+			(at 135.89 137.16 0)
 			(effects
 				(font
@@
 		)
 		(property "Description" "Power symbol creates a global label with name \"GND\" , ground"
-			(at 135.89 135.89 0)
+			(at 135.89 137.16 0)
 			(effects
 				(font
@@
 			)
 		)
-		(property "Footprint" ""
+		(property "Footprint" "Resistor_SMD:R_0805_2012Metric"
 			(at 60.452 146.05 90)
 			(effects
@@
 			)
 		)
-		(property "Footprint" ""
+		(property "Footprint" "Capacitor_SMD:C_0805_2012Metric"
 			(at 52.3748 153.67 0)
 			(effects
@@
 			)
 		)
-		(property "Footprint" ""
+		(property "Footprint" "Resistor_SMD:R_0805_2012Metric"
 			(at 121.666 51.054 90)
 			(effects
@@
 			)
 		)
-		(property "Footprint" ""
+		(property "Footprint" "Capacitor_SMD:C_0805_2012Metric"
 			(at 33.9852 104.14 0)
 			(effects
@@
 			)
 		)
-		(property "Footprint" ""
+		(property "Footprint" "Capacitor_SMD:C_0805_2012Metric"
 			(at 159.7152 156.21 0)
 			(effects
@@
 			)
 		)
-		(property "Footprint" ""
+		(property "Footprint" "Button_Switch_SMD:SW_SPDT_CK_JS102011SAQN"
 			(at 205.74 149.86 0)
 			(effects
@@
 			)
 		)
-		(property "Footprint" ""
+		(property "Footprint" "Resistor_SMD:R_0805_2012Metric"
 			(at 60.452 161.29 90)
 			(effects
@@
 			)
 		)
-		(property "Footprint" ""
+		(property "Footprint" "Connector_Dsub:DSUB-9_Socket_Horizontal_P2.77x2.84mm_EdgePinOffset9.40mm"
 			(at 29.21 154.94 0)
 			(effects
@@
 			)
 		)
-		(property "Footprint" ""
+		(property "Footprint" "Button_Switch_SMD:SW_SPDT_CK_JS102011SAQN"
 			(at 252.73 152.4 0)
 			(effects
@@
 			)
 		)
-		(property "Footprint" ""
+		(property "Footprint" "Button_Switch_SMD:SW_SPDT_CK_JS102011SAQN"
 			(at 252.73 137.16 0)
 			(effects
@@
 			)
 		)
-		(property "Footprint" ""
+		(property "Footprint" "Connector_Dsub:DSUB-9_Socket_Horizontal_P2.77x2.84mm_EdgePinOffset9.40mm"
 			(at 149.86 60.96 0)
 			(effects
@@
 			)
 		)
-		(property "Footprint" ""
+		(property "Footprint" "Capacitor_SMD:C_0805_2012Metric"
 			(at 16.8148 96.52 0)
 			(effects
@@
 			)
 		)
-		(property "Footprint" ""
+		(property "Footprint" "Capacitor_SMD:C_0805_2012Metric"
 			(at 117.8052 166.37 0)
 			(effects
@@
 			)
 		)
-		(property "Footprint" ""
+		(property "Footprint" "Capacitor_SMD:C_0805_2012Metric"
 			(at 103.8352 100.33 0)
 			(effects
@@
 			)
 		)
-		(property "Footprint" ""
+		(property "Footprint" "Capacitor_SMD:C_0805_2012Metric"
 			(at 97.4852 100.33 0)
 			(effects
@@
 			)
 		)
-		(property "Footprint" ""
+		(property "Footprint" "Button_Switch_SMD:SW_SPDT_CK_JS102011SAQN"
 			(at 252.73 121.92 0)
 			(effects

Commit message: lil hotfix
Parts:
- SW2: footprint (none) -> Button_Switch_SMD:SW_SPDT_CK_JS102011SAQN
Changed lines of the file:
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@@
 			)
 		)
-		(property "Footprint" ""
+		(property "Footprint" "Button_Switch_SMD:SW_SPDT_CK_JS102011SAQN"
 			(at 205.74 134.62 0)
 			(effects

Commit message: Hotfix for driver leds
Parts:
- J4: footprint (none) -> Connector_PinHeader_2.54mm:PinHeader_2x03_P2.54mm_Vertical
Changed lines of the file:
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@@
 			)
 		)
-		(property "Footprint" ""
+		(property "Footprint" "Connector_PinHeader_2.54mm:PinHeader_2x03_P2.54mm_Vertical"
 			(at 149.86 142.24 0)
 			(effects

Commit message: Pulsador Reset manual
Parts:
- added R14: 10k, Resistor_SMD:R_0805_2012Metric, symbol Device:R_US
- added SW1: SW_Push, Button_Switch_SMD:SW_Push_1P1T-SH_NO_CK_KMR2xxG, symbol Switch:SW_Push
Connections:
- net GND: now also SW1.2
- net MCLR: now also R14.2, SW1.1; no longer J4.1 (~{MCLR}/VPP)
- net VCC: now also R14.1
- no-connect marks 21 -> 22
Other:
- note added: "RESET MANUAL"

Commit message: Placa
Connections:
- net DRL_CTRL: now also U1.1 (RB9); no longer U1.2 (RC6)
- net HI_BEAM_CTRL: now also U1.5 (RC9); no longer U1.8 (RB10)
- net IN_LF: now also U1.15 (RB15); no longer U1.36 (RC3)
- net LF_FWD: now also U1.8 (RB10); no longer U1.9 (RB11)
- net LF_LIMIT: now also U1.34 (RA4); no longer U1.37 (RC4)
- net LF_REV: now also U1.9 (RB11); no longer U1.11 (RB13)
- net LIGHT_INT: now also U1.44 (RB8); no longer U1.13 (RA7)
- net LOW_BEAM_CTRL: now also U1.4 (RC8); no longer U1.5 (RC9)
- net SCL: now also U1.38 (RC5); no longer U1.44 (RB8)
- net SDA: now also U1.43 (RB7); no longer U1.1 (RB9)
- net TURN_LEFT_CTRL: now also U1.2 (RC6); no longer U1.3 (RC7)
- net TURN_RIGHT_CTRL: now also U1.3 (RC7); no longer U1.4 (RC8)
- net Usart1: now reaches U1.33 (RB4)
- net Usart1: now also J5.2
- net at U1.35 (RA9): no longer J5.2
Other:
- moved on the sheet: J5

Commit message: fin1
Connections:
- net IN_CA: now also U1.13 (RA7); no longer U1.26 (RC1)
- net IN_CR: now also U1.14 (RB14); no longer U1.27 (RC2)
- net LF_FWD: now also U1.37 (RC4); no longer U1.8 (RB10)
- net LF_LIMIT: now also U1.12 (RA10); no longer U1.34 (RA4)
- net LF_PWM: now also U1.35 (RA9); no longer U1.12 (RA10)
- net LF_REV: now also U1.36 (RC3); no longer U1.9 (RB11)
- net RXD: now also U1.23 (RB2); no longer U1.24 (RB3)
- net SCL: now also U1.41 (RB5); no longer U1.38 (RC5)
- net TXD: now also U1.24 (RB3); no longer U1.23 (RB2)
- net LedA: now reaches D2.1 (K), R11.1
- net CanH: now reaches J1.7, R12.1, U6.7 (CANH)
- net M: now reaches C3.2, R12.2, R13.1
- net Usart: now reaches J5.3, U1.32 (RA8)
- net Vbus: now reaches C2.1, U1.42 (VBUS)
- net Vcap: now reaches C13.2, U1.7 (VCAP)
- net CanL: now reaches J1.2, R13.2, U6.6 (CANL)

Commit message: a
Parts:
- R12, R13: footprint Resistor_SMD:R_0805_2012Metric -> Resistor_SMD:R_0603_1608Metric
Changed lines of the file:
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@@
 			)
 		)
-		(property "Footprint" "Resistor_SMD:R_0805_2012Metric"
+		(property "Footprint" "Resistor_SMD:R_0603_1608Metric"
 			(at 60.452 146.05 90)
 			(effects
@@
 			)
 		)
-		(property "Footprint" "Resistor_SMD:R_0805_2012Metric"
+		(property "Footprint" "Resistor_SMD:R_0603_1608Metric"
 			(at 60.452 161.29 90)
 			(effects
