File: KiCad/Transceptor_CAN.kicad_sch (KiCad schematic)
At the start: 26 parts, among them J1 DE9_Pins, J4 Conn_PIC_ICSP_ICD, J5 DE9_Pins, SW1 SW_Push, SW2 SW_SPDT, SW3 SW_SPDT, SW4 SW_SPDT, SW5 SW_SPDT, SW6 SW_SPDT, U1 PIC32MX250F128D-IPT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

Commit message: aaa
Parts:
- D2: footprint LED_SMD:LED_0805_2012Metric -> LED_SMD:LED_0805_2012Metric_Pad1.15x1.40mm_HandSolder
Changed lines of the file:
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@@
 			)
 		)
-		(property "Footprint" "LED_SMD:LED_0805_2012Metric"
+		(property "Footprint" "LED_SMD:LED_0805_2012Metric_Pad1.15x1.40mm_HandSolder"
 			(at 120.65 40.64 0)
 			(effects

Commit message: Finished
Other:
- company: (none) -> Marcel Lleonart, Eric Ruiz, Josep Leyva
Changed lines of the file:
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@@
 		(title "Procesament")
 		(date "2026-03-16")
+		(rev "28/04/2026")
+		(company "Marcel Lleonart, Eric Ruiz, Josep Leyva")
 	)
 	(text "MICROCONTROLADOR"
